File: eagle/Roland_140_ADSR_slim.sch (EAGLE design)
At the start: 60 parts, among them IC1 TL072P, Q1 BC557, Q2 BC557, Q3 BC557, T1 547, T10 547, T3 547, T4 547, T6 547, T7 547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

Commit message: routed and tweaked
Parts:
- added NORM: LSP10, solpad:LSP10
- GATE: value AUDIO-JACKERTHENVAR -> LSP10; device erthenvar:AUDIO-JACKERTHENVAR -> solpad:LSP10
- OUT: value AUDIO-JACKERTHENVAR -> AUDIO-JACKITEAD; device erthenvar:AUDIO-JACKERTHENVAR -> erthenvar:AUDIO-JACKITEAD
- R15, R16: device resistor:R-EU_0204_7 -> resistor:R-EU_0207_7
Connections:
- net GND: no longer GATE.RING
- net N$13: now also NORM.MP; no longer GATE.NORM
- net N$32: now also GATE.MP; no longer GATE.TIP
Other:
- moved on the sheet: OUT
Changed lines of the file:
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@@
 <part name="R14" library="resistor" deviceset="R-EU_" device="0204_7" value="100k"/>
 <part name="SUPPLY11" library="supply2" deviceset="GND" device=""/>
-<part name="R15" library="resistor" deviceset="R-EU_" device="0204_7" value="330r"/>
-<part name="R16" library="resistor" deviceset="R-EU_" device="0204_7" value="10k"/>
+<part name="R15" library="resistor" deviceset="R-EU_" device="0207_7" value="330r"/>
+<part name="R16" library="resistor" deviceset="R-EU_" device="0207_7" value="10k"/>
 <part name="SUPPLY12" library="supply2" deviceset="+12V" device=""/>
 <part name="R17" library="resistor" deviceset="R-EU_" device="0204_7" value="33k"/>
@@
 <part name="FB1" library="adafruit" deviceset="FB" device=""/>
 <part name="FB2" library="adafruit" deviceset="FB" device=""/>
-<part name="OUT" library="erthenvar" deviceset="AUDIO-JACK" device="ERTHENVAR" value="AUDIO-JACKERTHENVAR"/>
-<part name="GATE" library="erthenvar" deviceset="AUDIO-JACK" device="ERTHENVAR" value="AUDIO-JACKERTHENVAR"/>
+<part name="OUT" library="erthenvar" deviceset="AUDIO-JACK" device="ITEAD" value="AUDIO-JACKITEAD"/>
 <part name="DEC" library="pot" deviceset="3RP/1610N" device="" value="A1M"/>
 <part name="REL" library="pot" deviceset="3RP/1610N" device="" value="A1M"/>
 <part name="ATT" library="pot" deviceset="3RP/1610N" device="" value="A500K"/>
 <part name="SUST" library="pot" deviceset="3RP/1610N" device="" value="B100k"/>
+<part name="GATE" library="solpad" deviceset="LSP10" device=""/>
+<part name="NORM" library="solpad" deviceset="LSP10" device=""/>
 </parts>
 <sheets>
@@
 <attribute name="NAME" x="269.113" y="46.355" size="1.778" layer="95" rot="R180"/>
 </instance>
-<instance part="GATE" gate="G$1" x="58.42" y="45.72" smashed="yes" rot="MR180">
-<attribute name="NAME" x="50.927" y="41.275" size="1.778" layer="95" rot="MR180"/>
-</instance>
 <instance part="DEC" gate="G$1" x="200.66" y="15.24" rot="R90"/>
 <instance part="REL" gate="G$1" x="195.58" y="81.28" rot="R90"/>
 <instance part="ATT" gate="G$1" x="195.58" y="55.88" rot="R90"/>
 <instance part="SUST" gate="G$1" x="129.54" y="5.08"/>
+<instance part="GATE" gate="1" x="63.5" y="50.8" smashed="yes" rot="R90">
+<attribute name="NAME" x="60.579" y="49.53" size="1.778" layer="95" rot="R90"/>
+</instance>
+<instance part="NORM" gate="1" x="63.5" y="43.18" smashed="yes" rot="R90">
+<attribute name="NAME" x="60.579" y="36.83" size="1.778" layer="95" rot="R90"/>
+</instance>
 </instances>
 <busses>
@@
 <junction x="101.6" y="40.64"/>
 <pinref part="SUPPLY4" gate="GND" pin="GND"/>
-<wire x1="66.04" y1="43.18" x2="73.66" y2="43.18" width="0.1524" layer="91"/>
-<wire x1="73.66" y1="43.18" x2="73.66" y2="40.64" width="0.1524" layer="91"/>
-<wire x1="73.66" y1="40.64" x2="83.82" y2="40.64" width="0.1524" layer="91"/>
 <junction x="83.82" y="40.64"/>
-<pinref part="GATE" gate="G$1" pin="RING"/>
 </segment>
 <segment>
@@
 <pinref part="R3" gate="G$1" pin="1"/>
 <wire x1="66.04" y1="50.8" x2="73.66" y2="50.8" width="0.1524" layer="91"/>
-<pinref part="GATE" gate="G$1" pin="TIP"/>
+<pinref part="GATE" gate="1" pin="MP"/>
 </segment>
 </net>
@@
 <wire x1="45.72" y1="-2.54" x2="45.72" y2="20.32" width="0.1524" layer="91"/>
 <wire x1="45.72" y1="20.32" x2="68.58" y2="20.32" width="0.1524" layer="91"/>
-<wire x1="68.58" y1="20.32" x2="68.58" y2="45.72" width="0.1524" layer="91"/>
-<pinref part="GATE" gate="G$1" pin="NORM"/>
-<wire x1="68.58" y1="45.72" x2="66.04" y2="45.72" width="0.1524" layer="91"/>
-</segment>
-</net>
+<wire x1="68.58" y1="20.32" x2="68.58" y2="43.18" width="0.1524" layer="91"/>
+<wire x1="68.58" y1="43.18" x2="66.04" y2="43.18" width="0.1524" layer="91"/>
+<pinref part="NORM" gate="1" pin="MP"/>
+</segment>
+</net>
