File: eagle/Roland_140_ADSR_slim.sch (EAGLE design)
At the start: 61 parts, among them IC1 TL072P, Q1 BC557, Q2 BC557, Q3 BC557, T1 547, T10 547, T3 547, T4 547, T6 547, T7 547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

Commit message: added ground for gate input
Parts:
- added GND: LSP10, solpad:LSP10
Connections:
- net GND: now also GND.MP
Changed lines of the file:
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@@
 <part name="GATE" library="solpad" deviceset="LSP10" device=""/>
 <part name="NORM" library="solpad" deviceset="LSP10" device=""/>
+<part name="GND" library="solpad" deviceset="LSP10" device=""/>
+<part name="SUPPLY22" library="supply2" deviceset="GND" device=""/>
 </parts>
 <sheets>
@@
 <attribute name="NAME" x="60.579" y="36.83" size="1.778" layer="95" rot="R90"/>
 </instance>
+<instance part="GND" gate="1" x="63.5" y="60.96" smashed="yes" rot="R90">
+<attribute name="NAME" x="60.579" y="54.61" size="1.778" layer="95" rot="R90"/>
+</instance>
+<instance part="SUPPLY22" gate="GND" x="66.04" y="55.88"/>
 </instances>
 <busses>
@@
 <wire x1="86.36" y1="12.7" x2="63.5" y2="12.7" width="0.1524" layer="91"/>
 </segment>
+<segment>
+<pinref part="GND" gate="1" pin="MP"/>
+<pinref part="SUPPLY22" gate="GND" pin="GND"/>
+<wire x1="66.04" y1="60.96" x2="66.04" y2="58.42" width="0.1524" layer="91"/>
+</segment>
 </net>
